File: flight-pcb/flight-pcb.sch (KiCad schematic (older format))
At the start: 21 parts, among them J1 Conn_01x05, J2 Conn_01x06, J3 Conn_01x08, J4 Conn_01x20, J5 Conn_01x20, J6 Conn_01x05, J7 Conn_01x07, J8 Conn_01x02

Commit message: Update flight-pcb.sch
Parts:
- R1: value 68 -> 270
- R2: value 68 -> 309
- R3: value 68 -> 294
- R4: value 68 -> 100
Changed lines of the file:
@@
 U 1 1 62F58194
 P 5750 2200
-F 0 "R3" V 5750 2150 50  0000 C CNN
-F 1 "68" V 5750 2250 50  0000 C CNN
+F 0 "R3" V 5750 2200 50  0000 C CNN
+F 1 "294" V 5850 2200 50  0000 C CNN
 F 2 "Resistor_SMD:R_0603_1608Metric" V 5680 2200 50  0001 C CNN
 F 3 "~" H 5750 2200 50  0001 C CNN
@@
 U 1 1 62F604D5
 P 5750 2000
-F 0 "R2" V 5750 1950 50  0000 C CNN
-F 1 "68" V 5750 2050 50  0000 C CNN
+F 0 "R2" V 5750 2000 50  0000 C CNN
+F 1 "309" V 5850 2000 50  0000 C CNN
 F 2 "Resistor_SMD:R_0603_1608Metric" V 5680 2000 50  0001 C CNN
 F 3 "~" H 5750 2000 50  0001 C CNN
@@
 U 1 1 62F60DCD
 P 5750 1800
-F 0 "R1" V 5750 1750 50  0000 C CNN
-F 1 "68" V 5750 1850 50  0000 C CNN
+F 0 "R1" V 5750 1800 50  0000 C CNN
+F 1 "270" V 5850 1800 50  0000 C CNN
 F 2 "Resistor_SMD:R_0603_1608Metric" V 5680 1800 50  0001 C CNN
 F 3 "~" H 5750 1800 50  0001 C CNN
@@
 U 1 1 6305B3E4
 P 5750 2400
-F 0 "R4" V 5750 2350 50  0000 C CNN
-F 1 "68" V 5750 2450 50  0000 C CNN
+F 0 "R4" V 5750 2400 50  0000 C CNN
+F 1 "100" V 5850 2400 50  0000 C CNN
 F 2 "Resistor_SMD:R_0603_1608Metric" V 5680 2400 50  0001 C CNN
 F 3 "~" H 5750 2400 50  0001 C CNN
